File: pcb/rsdb_rev1.kicad_pcb (KiCad board)
At the start: 2 copper layers, 30 x 60 mm, 14 parts, among them J1 OLED_128x64, U1 MSM261DGT003, U2 MCU_Seeed_XIAO_RP2040

Commit message: final?
Parts:
- added G***: LOGO, LOGO, F.Cu at (75.1, 91.1)
- added G***: LOGO, LOGO, F.Cu at (75.0, 100.0)
- added G***: LOGO, LOGO, F.Cu at (61.5, 89.8)
- added G***: LOGO, LOGO, F.Cu at (88.5, 89.8)
- added G***: LOGO, RSdB:front, F.Cu at (39.8, 82.3)
- added REF**: OSHW-Symbol_6.7x6mm_SilkScreen, Symbol:OSHW-Symbol_6.7x6mm_SilkScreen, F.Cu at (79.8, 117.0)
- D1, D2: value ESD5Zxx -> PESD5V0F1BL; footprint Diode_SMD:D_SOD-523 -> Diode_SMD:D_0402_1005Metric_Pad0.77x0.64mm_HandSolder
- moved R1 1.02 mm to (77.9, 102.5), turned to 0 degrees
- moved R2 1.02 mm to (73.3, 102.5), turned to 180 degrees
- moved D1 0.14 mm to (62.9, 113.9)
- moved D2 0.14 mm to (66.9, 113.9)
Connections:
- R1 pad 2: Net-(U2-PA8_A4_D4_SDA) -> +3V3
- R2 pad 2: Net-(U2-PA9_A5_D5_SCL) -> +3V3
- U2 pad 5: Net-(U2-PA8_A4_D4_SDA) -> SDA
- U2 pad 6: Net-(U2-PA9_A5_D5_SCL) -> SCL
Routing:
- net +3V3: track 74.0 -> 109.6 mm
- net SCL: track 25.3 -> 29.8 mm
- net SDA: track 25.3 -> 29.8 mm
- net Net-(U2-PA9_A5_D5_SCL): track 2.65 -> 0.00 mm
- net Net-(U2-PA8_A4_D4_SDA): track 2.65 -> 0.00 mm
Other:
- board text added: "@cw-urn RSdB V1"
