File: pcb/rsdb_rev1.kicad_sch (KiCad schematic)
At the start: 10 parts, among them J1 OLED_128x64, U1 MSM261DGT003, U2 MCU_Seeed_XIAO_RP2040

Commit message: pcb
Parts:
- added H1, H2, H3, H4: MountingHole, MountingHole:MountingHole_2.2mm_M2, symbol Mechanical:MountingHole
- C1: footprint (none) -> Capacitor_SMD:C_0603_1608Metric_Pad1.08x0.95mm_HandSolder
- R1, R2, R3, R4: footprint (none) -> Resistor_SMD:R_0603_1608Metric_Pad0.98x0.95mm_HandSolder
- U2: footprint (none) -> ScottoKeebs_MCU:Seeed_XIAO_RP2040
Connections:
- net +3V3: now also C1.1, U1.1 (VDD)
- net GND: now also C1.2, U1.5 (GND), U1.6 (L/R)
Other:
- moved on the sheet: C1, D1, D2, J1, R1, R2, R3, R4, U1, U2

Commit message: final?
Parts:
- removed D1, D2: ESD5Zxx, Diode_SMD:D_SOD-523, symbol Diode:ESD5Zxx
- added D1, D2: PESD5V0F1BL, Diode_SMD:D_0402_1005Metric_Pad0.77x0.64mm_HandSolder, symbol rsdb:PESD5V0F1BL
Connections:
- net +3V3: now also R1.2, R2.2
- net GND: now also D1.2 (A2), D2.2 (A2)
- net SCL: now also U2.6 (PA9_A5_D5_SCL)
- net SDA: now also U2.5 (PA8_A4_D4_SDA)
- net at R3.1, U1.3 (DATA): now also D1.1 (A1)
- net at R4.1, U1.4 (CLK): now also D2.1 (A1)
Other:
- moved on the sheet: R1
